File: Martendo32.kicad_pcb (KiCad board)
At the start: 2 copper layers, 75.2 x 98.5 mm, 107 parts, among them CN2 ZX-MX1.25-2PWT, J1 AudioJack4_SwitchTR1, J2 Conn_01x03, J4 USB-C, Q1 NPN, Q2 AO3401A, SW1 SK-3296S-01-L3, U3 TP4056, U4 NS4168, U5 TPS61040DBV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

Commit message: Add files via upload
Parts:
- R14, R25: value 10K -> 1K
- R21: value 10K -> 33k
- R4: value 2K -> 5K1
- R5: value 2K -> 1K
- R6, R7: value 10K -> 5K1
- R8: value 10K -> 240R
Connections:
- J1 pad TN: /+3V3 -> Net-(U4-VOP)
- R111 pad 1: /+3V3 -> Net-(U4-VOP)
- R8 pad 1: /+3V3 -> Net-(U4-VOP)
- U4 pad 8: /+3V3 -> Net-(U4-VOP)
Routing:
- net Net-(U4-VOP): track 0.00 -> 30.9 mm, vias 0 -> 2
- net /+3V3: track 280.1 -> 265.5 mm, vias 7 -> 6
- net /HPJ+1: track 35.2 -> 32.6 mm
- net /SPK1-: track 41.4 -> 40.7 mm
- net GND: vias 128 -> 129

Commit message: Add files via upload
Routing:
- net /HPJ+1: track 32.6 -> 31.4 mm

Commit message: Add files via upload
Parts:
- moved LED1 59.7 mm to (118.0, 138.2)
- moved LED2 59.7 mm to (119.5, 138.2)
- moved R4 57.2 mm to (119.5, 134.8), turned to -90 degrees
- moved R5 55.6 mm to (117.8, 134.9), turned to -90 degrees
- moved C5 2.22 mm to (97.2, 64.3), turned to -90 degrees
- moved C6 0.93 mm to (98.8, 64.3), turned to -90 degrees
Routing:
- net Net-(LED2-C): track 69.1 -> 5.89 mm, vias 2 -> 0
- net Net-(LED1-C): track 66.8 -> 5.00 mm, vias 2 -> 0
- net +5V: track 242.0 -> 247.4 mm, vias 7 -> 8
- net /+3V3: track 265.5 -> 262.1 mm
- net Net-(LED2-A): track 3.77 -> 1.94 mm
- net /VIN: track 92.5 -> 93.4 mm
- net Net-(LED1-A): track 2.41 -> 1.76 mm
Other:
- board text added: "PCB v2.1 - 2026/02"
- board text added: "by Marius & Stephan B."
- board text removed: "PCB v2.0 - 2026/01"
- board text removed: "by Marius & Stephan Beha"

Commit message: Add files via upload
Parts:
- removed R24: 10K, KiCad_GB300-P4-SingleSided_SMT_V2:0603
- R20: value 10K -> 220K
- R21: value 33k -> 680K
Connections:
- C9 pad 1: +5V -> /+5VIN
- D1 pad 1: +5V -> /+5VIN
- J4 pad A4_B9: +5V -> /+5VIN
- J4 pad B4_A9: +5V -> /+5VIN
- Q2 pad 1: +5V -> /+5VIN
- R4 pad 1: +5V -> /+5VIN
- R5 pad 1: +5V -> /+5VIN
- U3 pad 4: +5V -> /+5VIN
- U3 pad 8: +5V -> /+5VIN
Routing:
- net +5V: track 247.4 -> 89.2 mm, vias 8 -> 2
- net /+5VIN: track 0.00 -> 131.1 mm, vias 0 -> 6

Commit message: Add files via upload
Parts:
- added J3: Conn_01x18_Socket, MOSER:687118183722, F.Cu at (100.2, 82.9)
- added REF**: BATT_CONN_SMT_292173, MOSER:BATT_CONN_SMT_292173, B.Cu at (110.6, 141.0)
- added X22: , , F.Cu at (96.5, 76.7)
- added X23: , , F.Cu at (96.4, 89.1)
Routing:
- net +5V: track 89.2 -> 63.5 mm, vias 2 -> 4
- net /TFT_RESET: track 22.4 -> 30.3 mm
- net /TFT_SPI_CLK: track 24.4 -> 31.9 mm
- net /TFT_CS: track 28.9 -> 35.9 mm
- net /TFT_SPI_MOSI: track 30.7 -> 37.6 mm
- net /+3V3: track 262.1 -> 268.9 mm
- net /TFT_SPI_MISO: track 32.6 -> 39.3 mm
- net /TFT_SPI_DC: track 27.0 -> 33.7 mm
- net /+5VIN: track 131.1 -> 136.6 mm
- net /KEY_RIGHT2: track 76.3 -> 74.2 mm
- net /BAT+: track 101.3 -> 103.0 mm
- net /KEY_SELECT1: track 80.8 -> 79.1 mm
- net /KEY_START1: track 91.9 -> 90.3 mm
- net /SD_DAT2: track 73.1 -> 74.6 mm
- net /UART0_TXD: track 54.5 -> 53.1 mm
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Other:
- outline, holes or cut-outs redrawn
- board text added: "PCB v2.2 - 2026/05"
- board text removed: "PCB v2.1 - 2026/02"

Commit message: Add files via upload
Other:
- outline, holes or cut-outs redrawn
Changed lines of the file:
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@@
 		)
 		(embedded_fonts no)
+		(model "Y:/KiCAD/3D/687118183722_Download_STP_687118183722_rev1.stp"
+			(offset
+				(xyz 0 0 0)
+			)
+			(scale
+				(xyz 1 1 1)
+			)
+			(rotate
+				(xyz 0 0 0)
+			)
+		)
 	)
 	(footprint "KiCad_GB300-P4-SingleSided_SMT_V2:0603"
@@
 		(layer "F.SilkS")
 	)
-	(gr_line
-		(start 46.59 149.578)
-		(end 46.59 100.578)
-		(stroke
-			(width 0.254)
-			(type default)
-		)
-		(layer "Edge.Cuts")
-	)
 	(gr_arc
 		(start 46.606 97.2276)
@@
 		(layer "Edge.Cuts")
 	)
-	(gr_arc
-		(start 48.59 151.578)
-		(mid 47.175786 150.992214)
-		(end 46.59 149.578)
+	(gr_line
+		(start 46.606 148.605)
+		(end 46.606 100.578)
 		(stroke
 			(width 0.254)
-			(type default)
+			(type solid)
 		)
 		(layer "Edge.Cuts")
 	)
-	(gr_line
-		(start 48.59 151.578)
-		(end 57.59 151.578)
+	(gr_arc
+		(start 49.606 151.605)
+		(mid 47.48468 150.72632)
+		(end 46.606 148.605)
 		(stroke
 			(width 0.254)
@@
 	)
 	(gr_line
-		(start 57.59 151.578)
-		(end 60.74 151.578)
+		(start 49.606 151.605)
+		(end 118.84 151.605)
 		(stroke
 			(width 0.254)
@@
 	)
 	(gr_line
-		(start 60.74 151.578)
-		(end 107.69 151.578)
-		(stroke
-			(width 0.254)
-			(type default)
-		)
-		(layer "Edge.Cuts")
-	)
-	(gr_line
 		(start 78.15 94.2276)
 		(end 49.606 94.2276)
@@
 	)
 	(gr_line
-		(start 84.79 53.078)
-		(end 84.8375 53.078)
-		(stroke
-			(width 0.254)
-			(type solid)
-		)
-		(layer "Edge.Cuts")
-	)
-	(gr_line
-		(start 84.8375 53.078)
-		(end 84.15 53.078)
-		(stroke
-			(width 0.254)
-			(type solid)
-		)
-		(layer "Edge.Cuts")
-	)
-	(gr_line
 		(start 102.19 53.078)
-		(end 84.8375 53.078)
+		(end 84.15 53.078)
 		(stroke
 			(width 0.254)
@@
 		(layer "Edge.Cuts")
 	)
-	(gr_line
-		(start 107.69 151.578)
-		(end 110.84 151.578)
-		(stroke
-			(width 0.254)
-			(type solid)
-		)
-		(layer "Edge.Cuts")
-	)
 	(gr_arc
 		(start 109.84 53.078)
@@
 		(layer "Edge.Cuts")
 	)
-	(gr_line
-		(start 119.84 151.578)
-		(end 110.84 151.578)
-		(stroke
-			(width 0.254)
-			(type default)
-		)
-		(layer "Edge.Cuts")
-	)
 	(gr_arc
-		(start 121.84 149.578)
-		(mid 121.254214 150.992214)
-		(end 119.84 151.578)
+		(start 121.84 148.605)
+		(mid 120.96132 150.72632)
+		(end 118.84 151.605)
 		(stroke
 			(width 0.254)
@@
 	)
 	(gr_line
-		(start 121.84 149.578)
+		(start 121.84 148.605)
 		(end 121.84 62.078)
 		(stroke
@@
 	)
 	(segment
-		(start 71.39 115.678)
-		(end 70.39 115.678)
+		(start 105.19 103.578)
+		(end 104.607 103.578)
 		(width 0.2)
 		(layer "F.Cu")
@@
 	)
 	(segment
-		(start 105.19 103.578)
-		(end 104.607 103.578)
-		(width 0.2)
+		(start 71.39 115.678)
+		(end 69.99 115.678)
+		(width 0.254)
 		(layer "F.Cu")
 		(net "/SD_CD")
@@
 	)
 	(segment
-		(start 71.591 117.9934)
-		(end 71.591 124.079)
-		(width 0.2)
-		(layer "B.Cu")
-		(net "/SD_CD")
-	)
-	(segment
 		(start 105.19 103.578)
 		(end 105.1424 103.6256)
@@
 	)
 	(segment
+		(start 69.99 115.678)
+		(end 69.99 115.6812)
+		(width 0.2)
+		(layer "B.Cu")
+		(net "/SD_CD")
+	)
+	(segment
 		(start 105.1424 103.6256)
 		(end 104.9424 103.6256)
@@
 	)
 	(segment
-		(start 70.19 115.678)
-		(end 70.59 116.078)
+		(start 71.59 117.833115)
+		(end 71.59 117.9924)
 		(width 0.2)
 		(layer "B.Cu")
@@
 	)
 	(segment
-		(start 69.99 115.678)
-		(end 70.19 115.678)
+		(start 103.391 111.179)
+		(end 105.091 112.879)
 		(width 0.2)
 		(layer "B.Cu")
@@
 	)
 	(segment
-		(start 103.391 111.179)
-		(end 105.091 112.879)
+		(start 71.591 124.079)
+		(end 73.99 126.478)
 		(width 0.2)
 		(layer "B.Cu")
@@
 	)
 	(segment
-		(start 70.59 116.078)
-		(end 70.59 116.833114)
+		(start 69.99 115.6812)
+		(end 70.59 116.2812)
 		(width 0.2)
 		(layer "B.Cu")
@@
 	)
 	(segment
-		(start 71.591 124.079)
-		(end 73.99 126.478)
+		(start 92.969271 129.2288)
+		(end 92.88047 129.3176)
 		(width 0.2)
 		(layer "B.Cu")
@@
 	)
 	(segment
-		(start 92.969271 129.2288)
-		(end 92.88047 129.3176)
+		(start 75.61323 128.098401)
+		(end 75.467229 127.9524)
 		(width 0.2)
 		(layer "B.Cu")
@@
 	)
 	(segment
-		(start 75.61323 128.098401)
-		(end 75.467229 127.9524)
+		(start 70.59 116.833114)
+		(end 71.59 117.833115)
 		(width 0.2)
 		(layer "B.Cu")
@@
 	)
 	(segment
-		(start 71.59 117.833115)
-		(end 71.59 117.9924)
+		(start 71.591 117.9934)
+		(end 71.591 124.079)
 		(width 0.2)
 		(layer "B.Cu")
@@
 	)
 	(segment
-		(start 70.59 116.833114)
-		(end 71.59 117.833115)
+		(start 70.59 116.2812)
+		(end 70.59 116.833114)
 		(width 0.2)
 		(layer "B.Cu")

Commit message: Add files via upload
Parts:
- added C12: 10uF, MOSER:0805, F.Cu at (69.8, 120.7)
- added R24: 10K, MOSER:0603, F.Cu at (112.8, 75.1)
- moved G*** 0.92 mm to (89.2, 144.3)
Connections:
- net Net-(U4-VOP) renamed /HPJ+
Routing:
- net /RP1_Y: track 30.1 -> 25.3 mm
- net /KEY_SELECT1: track 79.1 -> 81.3 mm
- net /KEY_START1: track 90.3 -> 92.5 mm
- net /RP1_X: track 51.8 -> 53.9 mm
- net /+5VIN: track 136.6 -> 137.7 mm
- net GND: vias 191 -> 194
