File: Martendo32.kicad_sch (KiCad schematic)
At the start: 100 parts, among them CN2 ZX-MX1.25-2PWT, J1 AudioJack4_SwitchTR1, J2 Conn_01x03, J4 USB-C, Q1 NPN, Q2 AO3401A, SW1 SK-3296S-01-L3, U3 TP4056, U4 NS4168, U5 TPS61040DBV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

Commit message: Add files via upload
added Analog Joysticks RP1/RP1
Parts:
- added RP1, RP2: Adafruit_2765, Martendo32Library:Adafruit_2765, symbol DoMiNi:Adafruit_2765_Mini_2-Axis_Analog_Thumbstick
Connections:
- net +3V3: now also RP1.X+, RP1.Y+, RP2.X+, RP2.Y+
- net GND: now also RP1.X-, RP1.Y-, RP2.X-, RP2.Y-
- net RP1_X: now reaches TP18.1, U1.32 (ESP_LDO_VO4)
- net RP1_X: now also RP1.X
- net RP1_Y: now reaches TP21.1, U1.33 (IO36)
- net RP1_Y: now also RP1.Y
- new net RP2_X: RP2.X
- new net RP2_Y: RP2.Y
Other:
- moved on the sheet: TP18, TP21

Commit message: Add files via upload
improved Silkscreen
Connections:
- net RP2_X: now also TP4.1, U1.60 (IO7)
- net RP2_Y: now also TP5.1, U1.59 (IO6)
Other:
- moved on the sheet: TP4, TP5
Changed lines of the file:
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@@
 	)
 	(junction
+		(at 63.5 20.32)
+		(diameter 0)
+		(color 0 0 0 0)
+	)
+	(junction
 		(at 334.01 146.05)
 		(diameter 0)
@@
 	)
 	(junction
+		(at 60.96 22.86)
+		(diameter 0)
+		(color 0 0 0 0)
+	)
+	(junction
 		(at 256.54 229.87)
 		(diameter 0)
@@
 	(wire
 		(pts
-			(xy 63.5 33.02) (xy 63.5 38.1)
+			(xy 63.5 19.05) (xy 63.5 20.32)
 		)
 		(stroke
@@
 	(wire
 		(pts
+			(xy 63.5 20.32) (xy 64.77 20.32)
+		)
+		(stroke
+			(width 0)
+			(type default)
+		)
+	)
+	(wire
+		(pts
 			(xy 215.9 231.14) (xy 227.33 231.14)
 		)
@@
 	(wire
 		(pts
+			(xy 60.96 22.86) (xy 60.96 38.1)
+		)
+		(stroke
+			(width 0)
+			(type default)
+		)
+	)
+	(wire
+		(pts
 			(xy 238.76 214.63) (xy 238.76 210.82)
 		)
@@
 	(wire
 		(pts
+			(xy 64.77 16.51) (xy 68.58 16.51)
+		)
+		(stroke
+			(width 0)
+			(type default)
+		)
+	)
+	(wire
+		(pts
 			(xy 251.46 257.81) (xy 264.16 257.81)
 		)
@@
 	(wire
 		(pts
-			(xy 60.96 33.02) (xy 60.96 38.1)
+			(xy 60.96 19.05) (xy 60.96 22.86)
 		)
 		(stroke
@@
 	(wire
 		(pts
+			(xy 63.5 20.32) (xy 63.5 38.1)
+		)
+		(stroke
+			(width 0)
+			(type default)
+		)
+	)
+	(wire
+		(pts
 			(xy 275.59 54.61) (xy 313.69 54.61)
 		)
@@
 	(wire
 		(pts
+			(xy 57.15 22.86) (xy 60.96 22.86)
+		)
+		(stroke
+			(width 0)
+			(type default)
+		)
+	)
+	(wire
+		(pts
 			(xy 236.22 74.93) (xy 237.49 74.93)
 		)
@@
 	(wire
 		(pts
+			(xy 64.77 20.32) (xy 64.77 16.51)
+		)
+		(stroke
+			(width 0)
+			(type default)
+		)
+	)
+	(wire
+		(pts
 			(xy 175.26 78.74) (xy 175.26 59.69)
 		)
@@
 		)
 	)
+	(label "RP2_Y"
+		(at 68.58 16.51 0)
+		(effects
+			(font
+				(size 1.27 1.27)
+			)
+			(justify left bottom)
+		)
+	)
 	(label "VIN"
 		(at 289.56 83.82 0)
@@
 		)
 	)
+	(label "RP2_X"
+		(at 57.15 22.86 0)
+		(effects
+			(font
+				(size 1.27 1.27)
+			)
+			(justify left bottom)
+		)
+	)
 	(label "ADC_VOLUME"
 		(at 332.74 240.03 0)
@@
 	(symbol
 		(lib_id "Connector:TestPoint")
-		(at 60.96 33.02 0)
+		(at 60.96 19.05 0)
 		(unit 1)
 		(exclude_from_sim no)
@@
 		(dnp no)
 		(property "Reference" "TP4"
-			(at 60.198 27.94 90)
+			(at 60.198 13.97 90)
 			(effects
 				(font
@@
 		)
 		(property "Value" "TestPoint"
-			(at 63.5 30.9879 0)
+			(at 63.5 17.0179 0)
 			(effects
 				(font
@@
 		)
 		(property "Footprint" "TestPoint:TestPoint_Pad_D1.0mm"
-			(at 66.04 33.02 0)
+			(at 66.04 19.05 0)
 			(effects
 				(font
@@
 		)
 		(property "Datasheet" "~"
-			(at 66.04 33.02 0)
+			(at 66.04 19.05 0)
 			(effects
 				(font
@@
 		)
 		(property "Description" "test point"
-			(at 60.96 33.02 0)
+			(at 60.96 19.05 0)
 			(effects
 				(font
@@
 	(symbol
 		(lib_id "Connector:TestPoint")
-		(at 63.5 33.02 0)
+		(at 63.5 19.05 0)
 		(unit 1)
 		(exclude_from_sim no)
@@
 		(dnp no)
 		(property "Reference" "TP5"
-			(at 62.738 27.94 90)
+			(at 62.738 13.97 90)
 			(effects
 				(font
@@
 		)
 		(property "Value" "TestPoint"
-			(at 66.04 30.9879 0)
+			(at 66.04 17.0179 0)
 			(effects
 				(font
@@
 		)
 		(property "Footprint" "TestPoint:TestPoint_Pad_D1.0mm"
-			(at 68.58 33.02 0)
+			(at 68.58 19.05 0)
 			(effects
 				(font
@@
 		)
 		(property "Datasheet" "~"
-			(at 68.58 33.02 0)
+			(at 68.58 19.05 0)
 			(effects
 				(font
@@
 		)
 		(property "Description" "test point"
-			(at 63.5 33.02 0)
+			(at 63.5 19.05 0)
 			(effects
 				(font

Commit message: Add files via upload
Parts:
- added R26: 10K, Resistor_SMD:R_0603_1608Metric_Pad0.98x0.95mm_HandSolder, symbol ESP32P4Gap-easyedapro:电阻
- added TP22, TP23: TestPoint, TestPoint:TestPoint_Pad_D1.0mm, symbol Connector:TestPoint
Connections:
- net KEY_FN1 is gone; now on net RP1_X: U1.51 (IO52)
- net KEY_L is gone; now on net RP1_Y: U1.52 (IO53)
- net KEY_R is gone; now on net RP2_X: U1.54 (IO54)
- net LCD_BACK: now also RP2.Y
- net RP1_X: no longer TP18.1, U1.32 (ESP_LDO_VO4)
- net RP1_Y: no longer TP21.1, U1.33 (IO36)
- net RP2_X: no longer TP4.1, U1.60 (IO7)
- net at Q1.2 (B), R13.1, R14.1: now also R26.1
- net LCD_BACK_ALT: now reaches TP13.1, U1.24 (IO28)
- net LCD_BACK_ALT: now also R26.2
- net at U1.16 (USB_DM): now also TP23.1
- net at U1.17 (USB_DP): now also TP22.1
- net RP2_Y: no longer names the net of TP5.1, U1.59 (IO6)
- net RP2_Y: no longer RP2.Y
- new net: TP21.1, U1.33 (IO36)
- new net: TP4.1, U1.60 (IO7)
- new net: TP18.1, U1.32 (ESP_LDO_VO4)
Other:
- note added: "Analog Joysticks (optional)"
- note added: "R26 is placed, if RP2 is used otherwise place only R14"
- moved on the sheet: RP1, RP2

Commit message: Add files via upload
Parts:
- R14, R25: value 10K -> 1K
- R21: value 10K -> 33k
- R4: value 2K -> 5K1
- R5: value 2K -> 1K
- R6, R7: value 10K -> 5K1
- R8: value 10K -> 240R
Connections:
- net +3V3: no longer J1.TN, R111.1, R8.1, U4.8 (VOP)
- new net: J1.TN, R111.1, R8.1, U4.8 (VOP)
Changed lines of the file:
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@@
 	)
 	(junction
+		(at 342.9 191.77)
+		(diameter 0)
+		(color 0 0 0 0)
+	)
+	(junction
 		(at 187.96 62.23)
 		(diameter 0)
@@
 	)
 	(junction
-		(at 355.6 212.09)
-		(diameter 0)
-		(color 0 0 0 0)
-	)
-	(junction
 		(at 363.22 146.05)
 		(diameter 0)
@@
 	)
 	(junction
-		(at 342.9 189.23)
-		(diameter 0)
-		(color 0 0 0 0)
-	)
-	(junction
 		(at 334.01 100.33)
 		(diameter 0)
@@
 	)
 	(junction
-		(at 355.6 207.01)
-		(diameter 0)
-		(color 0 0 0 0)
-	)
-	(junction
 		(at 227.33 231.14)
 		(diameter 0)
@@
 	)
 	(junction
-		(at 355.6 189.23)
-		(diameter 0)
-		(color 0 0 0 0)
-	)
-	(junction
 		(at 238.76 261.62)
 		(diameter 0)
@@
 	)
 	(junction
+		(at 356.87 191.77)
+		(diameter 0)
+		(color 0 0 0 0)
+	)
+	(junction
 		(at 231.14 114.3)
 		(diameter 0)
@@
 	(wire
 		(pts
-			(xy 349.25 212.09) (xy 355.6 212.09)
-		)
-		(stroke
-			(width 0)
-			(type default)
-		)
-	)
-	(wire
-		(pts
 			(xy 307.34 100.33) (xy 300.99 100.33)
 		)
@@
 	(wire
 		(pts
-			(xy 355.6 212.09) (xy 367.03 212.09)
+			(xy 349.25 212.09) (xy 367.03 212.09)
 		)
 		(stroke
@@
 	(wire
 		(pts
-			(xy 335.28 189.23) (xy 342.9 189.23)
-		)
-		(stroke
-			(width 0)
-			(type default)
-		)
-	)
-	(wire
-		(pts
 			(xy 34.29 250.19) (xy 44.45 250.19)
 		)
@@
 	(wire
 		(pts
+			(xy 370.84 184.15) (xy 373.38 184.15)
+		)
+		(stroke
+			(width 0)
+			(type default)
+		)
+	)
+	(wire
+		(pts
 			(xy 342.9 175.26) (xy 349.25 175.26)
 		)
@@
 	(wire
 		(pts
+			(xy 342.9 191.77) (xy 356.87 191.77)
+		)
+		(stroke
+			(width 0)
+			(type default)
+		)
+	)
+	(wire
+		(pts
 			(xy 153.67 265.43) (xy 152.4 265.43)
 		)
@@
 	(wire
 		(pts
+			(xy 356.87 191.77) (xy 356.87 207.01)
+		)
+		(stroke
+			(width 0)
+			(type default)
+		)
+	)
+	(wire
+		(pts
 			(xy 313.69 44.45) (xy 313.69 54.61)
 		)
@@
 	(wire
 		(pts
+			(xy 337.82 191.77) (xy 342.9 191.77)
+		)
+		(stroke
+			(width 0)
+			(type default)
+		)
+	)
+	(wire
+		(pts
 			(xy 100.33 175.26) (xy 106.68 175.26)
 		)
@@
 	(wire
 		(pts
-			(xy 335.28 189.23) (xy 335.28 180.34)
-		)
-		(stroke
-			(width 0)
-			(type default)
-		)
-	)
-	(wire
-		(pts
 			(xy 326.39 234.95) (xy 326.39 237.49)
 		)
@@
 	(wire
 		(pts
-			(xy 335.28 180.34) (xy 332.74 180.34)
+			(xy 332.74 180.34) (xy 337.82 180.34)
 		)
 		(stroke
@@
 	(wire
 		(pts
+			(xy 356.87 191.77) (xy 370.84 191.77)
+		)
+		(stroke
+			(width 0)
+			(type default)
+		)
+	)
+	(wire
+		(pts
 			(xy 153.67 245.11) (xy 149.86 245.11)
 		)
@@
 	(wire
 		(pts
-			(xy 342.9 189.23) (xy 355.6 189.23)
+			(xy 76.2 248.92) (xy 81.28 248.92)
 		)
 		(stroke
@@
 	(wire
 		(pts
-			(xy 76.2 248.92) (xy 81.28 248.92)
+			(xy 381 212.09) (xy 374.65 212.09)
 		)
 		(stroke
@@
 	(wire
 		(pts
-			(xy 381 212.09) (xy 374.65 212.09)
+			(xy 328.93 39.37) (xy 331.47 39.37)
 		)
 		(stroke
@@
 	(wire
 		(pts
-			(xy 328.93 39.37) (xy 331.47 39.37)
+			(xy 349.25 207.01) (xy 356.87 207.01)
 		)
 		(stroke
@@
 	(wire
 		(pts
-			(xy 342.9 189.23) (xy 342.9 186.69)
+			(xy 342.9 186.69) (xy 342.9 191.77)
 		)
 		(stroke
@@
 	(wire
 		(pts
-			(xy 373.38 184.15) (xy 373.38 189.23)
+			(xy 238.76 210.82) (xy 237.49 210.82)
 		)
 		(stroke
@@
 	(wire
 		(pts
-			(xy 238.76 210.82) (xy 237.49 210.82)
+			(xy 337.82 180.34) (xy 337.82 191.77)
 		)
 		(stroke
@@
 	(wire
 		(pts
-			(xy 349.25 207.01) (xy 355.6 207.01)
-		)
-		(stroke
-			(width 0)
-			(type default)
-		)
-	)
-	(wire
-		(pts
 			(xy 43.18 222.25) (xy 43.18 226.06)
 		)
@@
 	(wire
 		(pts
-			(xy 355.6 189.23) (xy 373.38 189.23)
-		)
-		(stroke
-			(width 0)
-			(type default)
-		)
-	)
-	(wire
-		(pts
 			(xy 201.93 220.98) (xy 190.5 220.98)
 		)
@@
 	(wire
 		(pts
-			(xy 355.6 207.01) (xy 360.68 207.01)
-		)
-		(stroke
-			(width 0)
-			(type default)
-		)
-	)
-	(wire
-		(pts
 			(xy 204.47 124.46) (xy 204.47 125.73)
 		)
@@
 	(wire
 		(pts
-			(xy 355.6 207.01) (xy 355.6 212.09)
+			(xy 377.19 146.05) (xy 391.16 146.05)
 		)
 		(stroke
@@
 	(wire
 		(pts
-			(xy 377.19 146.05) (xy 391.16 146.05)
+			(xy 116.84 83.82) (xy 120.65 83.82)
 		)
 		(stroke
@@
 	(wire
 		(pts
-			(xy 116.84 83.82) (xy 120.65 83.82)
+			(xy 100.33 182.88) (xy 100.33 180.34)
 		)
 		(stroke
@@
 	(wire
 		(pts
-			(xy 100.33 182.88) (xy 100.33 180.34)
+			(xy 342.9 175.26) (xy 342.9 176.53)
 		)
 		(stroke
@@
 	(wire
 		(pts
-			(xy 342.9 175.26) (xy 342.9 176.53)
+			(xy 370.84 191.77) (xy 370.84 184.15)
 		)
 		(stroke
@@
 	(wire
 		(pts
-			(xy 355.6 189.23) (xy 355.6 207.01)
-		)
-		(stroke
-			(width 0)
-			(type default)
-		)
-	)
-	(wire
-		(pts
 			(xy 226.06 60.96) (xy 226.06 57.15)
 		)
@@
 		)
 	)
-	(label "HPJ+"
-		(at 355.6 212.09 0)
-		(effects
-			(font
-				(size 1.2446 1.2446)
-			)
-			(justify left bottom)
-		)
-	)
 	(label "I2S_CTRL"
 		(at 96.52 29.21 90)
@@
 			)
 		)
-		(property "Value" "10K"
+		(property "Value" "5K1"
 			(at 322.326 40.132 0)
 			(effects
@@
 			)
 		)
-		(property "Value" "10K"
+		(property "Value" "1K"
 			(at 85.09 187.198 0)
 			(effects
@@
 			)
 		)
-		(property "Value" "2K"
+		(property "Value" "1K"
 			(at 241.554 61.722 0)
 			(effects
@@
 			)
 		)
-		(property "Value" "10K"
+		(property "Value" "1K"
 			(at 366.522 168.402 0)
 			(effects
@@
 			)
 		)
-		(property "Value" "10K"
+		(property "Value" "5K1"
 			(at 255.778 30.988 0)
 			(effects
@@
 			)
 		)
-		(property "Value" "2K"
+		(property "Value" "5K1"
 			(at 241.046 75.692 0)
 			(effects
@@
 			)
 		)
-		(property "Value" "10K"
+		(property "Value" "33k"
 			(at 333.248 88.392 0)
 			(effects
@@
 			)
 		)
-		(property "Value" "10K"
+		(property "Value" "240R"
 			(at 372.872 177.546 0)
 			(effects

Commit message: Add files via upload
Parts:
- R20: value 10K -> 220K
- R21: value 33k -> 680K
Connections:
- net +5V: no longer C9.1, D1.1 (A), J4.A4_B9 (VBUS_A), J4.B4_A9 (VBUS_B), Q2.1 (G), R24.1, R4.1, R5.1, U3.4 (VCC), U3.8 (CE)
- new net +5VIN: C9.1, D1.1 (A), J4.A4_B9 (VBUS_A), J4.B4_A9 (VBUS_B), Q2.1 (G), R24.1, R4.1, R5.1, U3.4 (VCC), U3.8 (CE)

Commit message: Add files via upload
Parts:
- added J3: Conn_01x18_Socket, MOSER:687118183722, symbol Connector:Conn_01x18_Socket
- LED1, LED2, SD1, U1: value ~ -> (none)
Connections:
- net +3V3: now also J3.10 (Pin_10), J3.9 (Pin_9)
- net GND: now also J3.1 (Pin_1), J3.8 (Pin_8)
- net TFT_CS: now also J3.5 (Pin_5)
- net TFT_RESET: now also J3.2 (Pin_2)
- net TFT_SPI_CLK: now also J3.3 (Pin_3)
- net TFT_SPI_DC: now also J3.4 (Pin_4)
- net TFT_SPI_MISO: now also J3.7 (Pin_7)
- net TFT_SPI_MOSI: now also J3.6 (Pin_6)
- net at LCD1.11 (Pin_11), R12.2: now also J3.11 (Pin_11)
- net at LCD1.12 (Pin_12), R11.2: now also J3.12 (Pin_12)
- net at LCD1.13 (Pin_13), R10.2: now also J3.13 (Pin_13)
- net at LCD1.14 (Pin_14), R9.2: now also J3.14 (Pin_14)
Other:
- moved on the sheet: H1, H2, LCD1, Q1, R10, R11, R12, R13, R14, R26, R8, R9

Commit message: Add files via upload
Parts:
- added C12: 10uF, MOSER:0805, symbol ESP32P4Gap-easyedapro:Capacitance
- R24: footprint KiCad_GB300-P4-SingleSided_SMT_V2:0603 -> MOSER:0603
Connections:
- net +5V: now also C12.1
- net GND: now also C12.2
- net HPJ+: now also J1.TN, R111.1, R8.1, U4.8 (VOP)
Changed lines of the file:
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@@
 	)
 	(junction
+		(at 157.48 41.91)
+		(diameter 0)
+		(color 0 0 0 0)
+	)
+	(junction
 		(at 191.77 213.36)
 		(diameter 0)
@@
 	(wire
 		(pts
+			(xy 157.48 41.91) (xy 267.97 41.91)
+		)
+		(stroke
+			(width 0)
+			(type default)
+		)
+	)
+	(wire
+		(pts
 			(xy 326.39 234.95) (xy 326.39 237.49)
 		)
@@
 	(wire
 		(pts
-			(xy 125.73 41.91) (xy 267.97 41.91)
+			(xy 125.73 41.91) (xy 157.48 41.91)
 		)
 		(stroke
@@
 	(wire
 		(pts
+			(xy 157.48 52.07) (xy 157.48 55.88)
+		)
+		(stroke
+			(width 0)
+			(type default)
+		)
+	)
+	(wire
+		(pts
 			(xy 63.5 106.68) (xy 63.5 110.49)
 		)
@@
 	)
 	(label "HPJ+"
-		(at 373.38 189.23 0)
+		(at 370.84 191.77 0)
 		(effects
 			(font
@@
 	)
 	(symbol
+		(lib_id "ESP32P4Gap-easyedapro:Capacitance")
+		(at 157.48 46.99 270)
+		(unit 1)
+		(body_style 1)
+		(exclude_from_sim no)
+		(in_bom yes)
+		(on_board yes)
+		(in_pos_files yes)
+		(dnp no)
+		(property "Reference" "C12"
+			(at 162.56 48.26 90)
+			(show_name no)
+			(do_not_autoplace no)
+			(effects
+				(font
+					(size 1.2446 1.2446)
+				)
+				(justify right top)
+			)
+		)
+		(property "Value" "10uF"
+			(at 162.56 43.18 90)
+			(show_name no)
+			(do_not_autoplace no)
+			(effects
+				(font
+					(size 1.2446 1.2446)
+				)
+				(justify right top)
+			)
+		)
+		(property "Footprint" "MOSER:0805"
+			(at 157.48 46.99 0)
+			(hide yes)
+			(show_name no)
+			(do_not_autoplace no)
+			(effects
+				(font
+					(size 1.27 1.27)
+				)
+			)
+		)
+		(property "Datasheet" ""
+			(at 157.48 46.99 0)
+			(hide yes)
+			(show_name no)
+			(do_not_autoplace no)
+			(effects
+				(font
+					(size 1.27 1.27)
+				)
+			)
+		)
+		(property "Description" ""
+			(at 157.48 46.99 0)
+			(hide yes)
+			(show_name no)
+			(do_not_autoplace no)
+			(effects
+				(font
+					(size 1.27 1.27)
+				)
+			)
+		)
+		(pin "1"
+		)
+		(pin "2"
+		)
+		(instances
+			(project "Martendo32"
+				(path "/4d50824d-5e8b-40d1-81c7-e2bd3d54a2c4"
+					(reference "C12")
+					(unit 1)
+				)
+			)
+		)
+	)
+	(symbol
 		(lib_id "Connector:TestPoint")
 		(at 58.42 110.49 180)
@@
 	)
 	(symbol
+		(lib_id "ESP32P4Gap-easyedapro:Ground-GND")
+		(at 157.48 55.88 0)
+		(unit 1)
+		(body_style 1)
+		(exclude_from_sim no)
+		(in_bom yes)
+		(on_board yes)
+		(in_pos_files yes)
+		(dnp no)
+		(property "Reference" "#PWR0158"
+			(at 157.48 55.88 0)
+			(hide yes)
+			(show_name no)
+			(do_not_autoplace no)
+			(effects
+				(font
+					(size 1.27 1.27)
+				)
+			)
+		)
+		(property "Value" "GND"
+			(at 157.48 55.88 0)
+			(hide yes)
+			(show_name no)
+			(do_not_autoplace no)
+			(effects
+				(font
+					(size 1.5748 1.5748)
+				)
+			)
+		)
+		(property "Footprint" "ESP32P4Gap-easyedapro:"
+			(at 157.48 55.88 0)
+			(hide yes)
+			(show_name no)
+			(do_not_autoplace no)
+			(effects
+				(font
+					(size 1.27 1.27)
+				)
+			)
+		)
+		(property "Datasheet" ""
+			(at 157.48 55.88 0)
+			(hide yes)
+			(show_name no)
+			(do_not_autoplace no)
+			(effects
+				(font
+					(size 1.27 1.27)
+				)
+			)
+		)
+		(property "Description" ""
+			(at 157.48 55.88 0)
+			(hide yes)
+			(show_name no)
+			(do_not_autoplace no)
+			(effects
+				(font
+					(size 1.27 1.27)
+				)
+			)
+		)
+		(pin "1"
+		)
+		(instances
+			(project "Martendo32"
+				(path "/4d50824d-5e8b-40d1-81c7-e2bd3d54a2c4"
+					(reference "#PWR0158")
+					(unit 1)
+				)
+			)
+		)
+	)
+	(symbol
 		(lib_id "ESP32P4Gap-easyedapro:TS-1187A-B-A-B")
 		(at 196.85 267.97 0)
@@
 			)
 		)
-		(property "Footprint" "KiCad_GB300-P4-SingleSided_SMT_V2:0603"
+		(property "Footprint" "MOSER:0603"
 			(at 264.16 119.38 0)
 			(hide yes)

Commit message: added value to U1
Parts:
- U1: value (none) -> WT0132P4A1N16R32
Changed lines of the file:
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@@
 			)
 		)
-		(property "Value" ""
-			(at 78.74 73.66 0)
+		(property "Value" "WT0132P4A1N16R32"
+			(at 77.978 76.962 0)
 			(show_name no)
 			(do_not_autoplace no)
@@
 			)
 		)
-		(property "Description" ""
+		(property "Description" "WT0132P4A1N16R32"
 			(at 78.74 73.66 0)
 			(hide yes)
